File: CommRF/PN715001A/PN715001A.sch (KiCad schematic (older format))
At the start: 50 parts, among them J1 PWR +3.3V, J2 HEADER_1x02, J3 HEADER_2x05_PARALLEL, J4 HEADER_2x03_PARALLEL, P1 ANTENNA, P4 CONN_01X01, P5 CONN_01X01, P6 CONN_01X01, P7 CONN_01X01, U1 PN7150, Y1 NX2016HA

Commit message: NFC-Reader
Parts:
- added R3: 47k, Resistors_SMD:R_0603, symbol R
- D1: symbol LED -> LED-RESCUE-PN715001A
- J1: value PWR +3.3V -> VBAT +5V
Connections:
- wire segments 122 -> 126
Changed lines of the file:
@@
 EESchema Schematic File Version 2
+LIBS:PN715001A-rescue
 LIBS:power
 LIBS:device
@@
 LIBS:MLAB_U
 LIBS:PN715001A-cache
-EELAYER 25 0
+EELAYER 26 0
 EELAYER END
 $Descr A4 11693 8268
@@
 P 1950 6650
 F 0 "J1" H 1600 6850 50  0000 C CNN
-F 1 "PWR +3.3V" V 1950 6700 40  0001 C CNN
+F 1 "VBAT +5V" V 1950 6700 40  0001 C CNN
 F 2 "Mlab_Pin_Headers:Straight_2x03" H 1950 6650 60  0001 C CNN
 F 3 "" H 1950 6650 60  0000 C CNN
@@
 $EndComp
 $Comp
-L LED D1
+L LED-RESCUE-PN715001A D1
 U 1 1 5939E943
 P 4450 1400
@@
 	1    0    0    -1
 $EndComp
+$Comp
+L R R3
+U 1 1 59411BA4
+P 3100 3700
+F 0 "R3" V 3180 3700 50  0000 C CNN
+F 1 "47k" V 3100 3700 50  0000 C CNN
+F 2 "Resistors_SMD:R_0603" V 3030 3700 50  0001 C CNN
+F 3 "" H 3100 3700 50  0000 C CNN
+	1    3100 3700
+	1    0    0    -1
+$EndComp
+Text Label 2800 3650 0    60   ~ 0
+VBAT
+Wire Wire Line
+	3100 3550 3100 3500
+Connection ~ 3100 3500
+Wire Wire Line
+	3100 3850 3100 3900
+Wire Wire Line
+	3100 3900 2800 3900
+Wire Wire Line
+	2800 3900 2800 3650
 $EndSCHEMATC
