File: Clock/NixieClock01A/NixieClock01A/NixieClock01A.sch (KiCad schematic (older format))
At the start: 17 parts, among them U1 74141, U2 PCF8574, U3 ESP-12E

Commit message: LM3478
Parts:
- added C?: C, Capacitor_SMD:C_0603_1608Metric, symbol Device:C
- added C? (x2): 22n, Capacitor_SMD:C_0603_1608Metric, symbol Device:C
- added C? (x2): 10u, Capacitor_SMD:C_0805_2012Metric, symbol Device:C
- added D?: D_Schottky, symbol Device:D_Schottky
- added L?: L_Core_Ferrite, symbol Device:L_Core_Ferrite
- added Q?: Q_NMOS_DSG, symbol Device:Q_NMOS_DSG
- added R? (x4): R, Resistor_SMD:R_0603_1608Metric, symbol Device:R
- added R?: 4k7, Resistor_SMD:R_0603_1608Metric, symbol Device:R
- added R?: 40k, Resistor_SMD:R_0603_1608Metric, symbol Device:R
- added R? (x3): R, Resistor_SMD:R_0805_2012Metric, symbol Device:R
- added U?: LM3478, symbol lm3478:LM3478
Connections:
- net labels added: Uanode, VCC
- wire segments 42 -> 103

Commit message: LM3478, ESP8266 layout
Parts:
- removed Q?: Q_NMOS_DSG, symbol Device:Q_NMOS_DSG
- added C11, C12: 100n, Capacitor_SMD:C_0603_1608Metric, symbol Device:C
- added C13: 1u, Capacitor_SMD:C_2220_5650Metric, symbol Device:C
- added C14: 100u, Capacitor_Tantalum_SMD:CP_EIA-7343-31_Kemet-D, symbol Device:CP
- added C15, C16: 10u, Capacitor_SMD:C_0805_2012Metric, symbol Device:C
- added D2: WS2812B, LED_SMD:LED_WS2812B_PLCC4_5.0x5.0mm_P3.2mm, symbol LED:WS2812B
- added J1: Conn_01x06_Male, Connector_PinHeader_2.54mm:PinHeader_1x06_P2.54mm_Vertical, symbol Connector:Conn_01x06_Male
- added N1: ZM1080, zm1080:ZM1080, symbol mynixies:ZM1080
- added Q1: Q_NMOS_GDS, Package_TO_SOT_SMD:TO-252-2, symbol Device:Q_NMOS_GDS
- C9: renamed from C?; value 10u -> 100n; footprint Capacitor_SMD:C_0805_2012Metric -> Capacitor_SMD:C_1206_3216Metric
- D1: renamed from D?; footprint (none) -> Diode_SMD:D_SMB
- L1: renamed from L?; footprint (none) -> Inductor_SMD:L_Wuerth_WE-PD-Typ-LS_Handsoldering
- U4: renamed from U?; footprint (none) -> Package_SO:SO-8_5.3x6.2mm_P1.27mm
- gave numbers to parts that had none: 13
Connections:
- net labels added: NeoPix1, RX, TX
- wire segments 103 -> 132
- no-connect marks 0 -> 3

Commit message: Nixie layout
Parts:
- added C17, C18, C19, C20, C21, C22, C23, C24, C27, C28, C29, C30, C31, C32: 100n, Capacitor_SMD:C_0603_1608Metric, symbol Device:C
- added C25, C26: 10u, Capacitor_SMD:C_0805_2012Metric, symbol Device:C
- added D3, D4, D5, D6, D7: WS2812B, LED_SMD:LED_WS2812B_PLCC4_5.0x5.0mm_P3.2mm, symbol LED:WS2812B
- added J2, J3: Conn_02x16_Odd_Even, Connector_PinSocket_2.54mm:PinSocket_2x16_P2.54mm_Vertical, symbol Connector_Generic:Conn_02x16_Odd_Even
- added N2, N3, N4, N5, N6: ZM1080, riske-lib:ZM1080, symbol mynixies:ZM1080
- added R19, R20: R, Resistor_SMD:R_0603_1608Metric, symbol Device:R
- added R21, R22, R23, R24, R25, R26: 27k, Resistor_SMD:R_1206_3216Metric, symbol Device:R
- added U10: L78L33_TO92, Package_TO_SOT_THT:TO-92_Inline, symbol Regulator_Linear:L78L33_TO92
- added U11, U12, U13, U5, U8: 74141, Package_DIP:DIP-16_W7.62mm, symbol 74xx_IEEE:74141
- added U6, U7: PCF8574, Package_SO:SOIC-16W_5.3x10.2mm_P1.27mm, symbol Interface_Expansion:PCF8574
- added U9: L78L05_TO92, Package_TO_SOT_THT:TO-92_Inline, symbol Regulator_Linear:L78L05_TO92
- C13: value 1u -> 1u/200V
- C9: value 100n -> 100n/200V
- N1: footprint zm1080:ZM1080 -> riske-lib:ZM1080
- U2: footprint Package_DIP:DIP-16_W7.62mm -> Package_SO:SOIC-16W_5.3x10.2mm_P1.27mm
Connections:
- net labels added: C1, C2, C3, C4, D1, D2, D3, D4, E1, E2, E3, E4, F1, F2, F3, F4, NeoPix
- net labels removed: NeoPix1
- wire segments 132 -> 323
- no-connect marks 3 -> 15
