File: Clock/NixieClock01A/NixieClock01A.kicad_pcb (KiCad board)
At the start: 2 copper layers, 97 parts, among them J1 Conn_01x06_Male, J10 Conn_01x01_Male, J11 Conn_01x01_Male, J12 Conn_01x01_Male, J2 Conn_02x16_Odd_Even, J3 Conn_02x16_Odd_Even, J4 USB_B_Micro, J5 Conn_01x01_Male, J6 Conn_01x01_Male, J7 Conn_01x01_Male, J8 Conn_01x01_Male, J9 Conn_01x01_Male, Q1 Q_NMOS_GDS, U1 74141, U11 74141, U12 74141, U13 74141, U2 PCF8574, U3 ESP-12E, U4 LM3478, U5 74141, U6 PCF8574, U7 PCF8574, U8 74141, U9 TC1262-33

Commit message: Final
Parts:
- added G***: LOGO, riske-lib:LogoGalaxy15x15, F.Cu at (107.5, 114.3)
- added G***: LOGO, riske-lib:LogoGalaxy15x15, F.Cu at (206.5, 101.0)
- added J13: Conn_01x02_Male, Connector_PinHeader_2.54mm:PinHeader_1x02_P2.54mm_Vertical, F.Cu at (227.1, 59.0)
- added J14: Conn_01x04_Male, Connector_PinSocket_2.54mm:PinSocket_1x04_P2.54mm_Vertical, F.Cu at (202.1, 59.6)
- added LA1: Lamp_Neon, Package_TO_SOT_THT:TO-92, F.Cu at (190.8, 141.9)
- added LA2: Lamp_Neon, Package_TO_SOT_THT:TO-92, F.Cu at (138.5, 141.9)
- added R27: 1M, Resistor_SMD:R_1206_3216Metric, B.Cu at (193.4, 136.8)
- added R28: 1M, Resistor_SMD:R_1206_3216Metric, B.Cu at (190.7, 136.8)
- added R29: 1M, Resistor_SMD:R_1206_3216Metric, B.Cu at (138.5, 136.7)
- added R30: 1M, Resistor_SMD:R_1206_3216Metric, B.Cu at (141.1, 136.7)
- added R31: 4K7, Resistor_SMD:R_0603_1608Metric, F.Cu at (234.3, 93.6)
- added R32: 4K7, Resistor_SMD:R_0603_1608Metric, F.Cu at (234.3, 91.9)
- R7: value 220k -> 330k
- U3: footprint RF_Module:ESP-12E -> riske-lib:ESP-12E
- moved R7 31.1 mm to (233.6, 65.4), turned to 0 degrees
- moved R5 28.6 mm to (238.8, 67.0), turned to 180 degrees
- moved C3 27.2 mm to (238.8, 68.8), turned to 180 degrees
- moved R8 26.8 mm to (233.6, 67.1), turned to 180 degrees
- moved R9 26.0 mm to (238.8, 70.6), turned to 180 degrees
- moved R2 22.9 mm to (231.9, 91.9), turned to 270 degrees
- moved R4 21.3 mm to (235.0, 70.6), turned to 180 degrees
- moved R3 21.3 mm to (229.7, 91.9), turned to 270 degrees
- moved U3 19.8 mm to (236.3, 80.9), turned to 270 degrees
- moved R6 18.6 mm to (226.9, 91.2), turned to 180 degrees
- moved J1 9.63 mm to (217.0, 74.7), turned to 0 degrees
- moved C5 8.95 mm to (221.2, 72.6), turned to 180 degrees
- moved U9 6.21 mm to (132.5, 64.5), turned to 0 degrees
- moved C26 4.75 mm to (126.9, 62.8), turned to 270 degrees
- moved C4 2.84 mm to (221.0, 77.4), turned to 270 degrees
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Connections:
- R7 pad 1: +3V3 -> /ADC-IN
- U3 pad 7: Net-(U3-Pad7) -> /NeoPix
- U9 pad 4: (no net) -> GND
Routing:
- net /NeoPix: track 85.3 -> 169.3 mm
- net /SCL: track 63.5 -> 106.4 mm
- net /SDA: track 63.4 -> 105.5 mm
- net +3V3: track 158.8 -> 197.6 mm
- net /Uanode: track 292.2 -> 304.1 mm
- net +5V: track 440.8 -> 430.3 mm
- net GND: track 72.9 -> 82.7 mm, vias 39 -> 53
- net /ADC-IN: track 0.00 -> 8.12 mm
- net Net-(LA1-Pad3): track 0.00 -> 3.91 mm
- net Net-(LA1-Pad1): track 0.00 -> 3.81 mm
- net Net-(LA2-Pad3): track 0.00 -> 3.80 mm
- net Net-(LA2-Pad1): track 0.00 -> 3.80 mm
- net /ADC: track 10.7 -> 14.0 mm
- net Net-(N6-Pad8): track 19.7 -> 22.0 mm
- net Net-(N4-Pad2): track 54.1 -> 56.0 mm
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Other:
- board outline added: 150 x 102 mm
- board text added: "NixieClock01A"
