File: Clock/NixieClock01A/NixieClock01A.sch (KiCad schematic (older format))
At the start: 89 parts, among them J1 Conn_01x06_Male, J2 Conn_02x16_Odd_Even, J3 Conn_02x16_Odd_Even, Q1 Q_NMOS_GDS, U1 74141, U10 L78L33_TO92, U11 74141, U12 74141, U13 74141, U2 PCF8574, U3 ESP-12E, U4 LM3478, U5 74141, U6 PCF8574, U7 PCF8574, U8 74141, U9 L78L05_TO92

Commit message: Power supplies layout
Parts:
- removed C16, C25, C4: 10u, Capacitor_SMD:C_0805_2012Metric, symbol Device:C
- removed C29: 100n, Capacitor_SMD:C_0603_1608Metric, symbol Device:C
- removed U10: L78L33_TO92, Package_TO_SOT_THT:TO-92_Inline, symbol Regulator_Linear:L78L33_TO92
- removed U9: L78L05_TO92, Package_TO_SOT_THT:TO-92_Inline, symbol Regulator_Linear:L78L05_TO92
- added C16, C4: TPSC107K010R0075, Capacitor_Tantalum_SMD:CP_EIA-6032-28_Kemet-C, symbol Device:CP
- added D8: D_TVS, Diode_SMD:D_SMC, symbol Device:D_TVS
- added F1: Fuse, Fuse:Fuse_1206_3216Metric, symbol Device:Fuse
- added J10, J11, J12, J5, J6, J7, J8, J9: Conn_01x01_Male, MountingHole:MountingHole_3.2mm_M3_DIN965_Pad, symbol Connector:Conn_01x01_Male
- added J4: USB_B_Micro, Connector_USB:USB_Micro-B_Molex-105017-0001, symbol Connector:USB_B_Micro
- added U9: TC1262-33, Package_TO_SOT_SMD:SOT-223, symbol Regulator_Linear:TC1262-33
- C15: value 10u -> 100n; footprint Capacitor_SMD:C_0805_2012Metric -> Capacitor_SMD:C_0603_1608Metric
- C30: value 100n -> 1u
Connections:
- wire segments 323 -> 345
- no-connect marks 15 -> 18

Commit message: Final
Parts:
- added J13: Conn_01x02_Male, Connector_PinHeader_2.54mm:PinHeader_1x02_P2.54mm_Vertical, symbol Connector:Conn_01x02_Male
- added J14: Conn_01x04_Male, Connector_PinSocket_2.54mm:PinSocket_1x04_P2.54mm_Vertical, symbol Connector:Conn_01x04_Male
- added LA1, LA2: Lamp_Neon, Package_TO_SOT_THT:TO-92, symbol Device:Lamp_Flash
- added R27, R28, R29, R30: 1M, Resistor_SMD:R_1206_3216Metric, symbol Device:R
- added R31, R32: 4K7, Resistor_SMD:R_0603_1608Metric, symbol Device:R
- R7: value 220k -> 330k
- U3: footprint RF_Module:ESP-12E -> riske-lib:ESP-12E
Connections:
- net labels added: ADC-IN
- wire segments 345 -> 392
- no-connect marks 18 -> 27
